File: hardware/mainboard/mainboard.kicad_sch (KiCad schematic)
At the start: 16 parts, among them J1 LEG1_RJ11, J2 LEG2_RJ11, J3 LEG3_RJ11, J4 LEG4_RJ11, J5 LEG5_RJ11, J6 LEG6_RJ11, J7 SBEC_5V_IN, J9 IMU_I2C, U1 ESP32-WROOM-32D, U2 SP3485CN

Commit message: hardware: restore R1 bus termination value to 100R
mainboard_sch.py already specified 100R for the RS485 bus termination
resistor (R1), but the committed mainboard.kicad_sch still had the old
120R value — it hadn't been regenerated before the V1/V2 restructuring,
and my earlier revert (to undo an accidental test-regeneration) put the
stale 120R value back instead of the intended 100R. Confirmed against
diff.txt (the pre-migration pending diff) and regenerated from source;
no other change.

Co-Authored-By: Claude Sonnet 5 <noreply@anthropic.com>
Parts:
- R1: value 120 -> 100
Changed lines of the file:
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@@
 			)
 		)
-		(property "Value" "120"
+		(property "Value" "100"
 			(at 220 98.81 0)
 			(effects
